Commit message: Testing URDF loading.

File: models/iiwa/model.urdf (robot description, URDF)
Before this commit: robot lbr_iiwa, 8 links, 7 joints
Links:
- removed link lbr_iiwa_link_3
- removed link lbr_iiwa_link_4
- removed link lbr_iiwa_link_5
- removed link lbr_iiwa_link_6
- removed link lbr_iiwa_link_7
Joints:
- removed joint lbr_iiwa_joint_3
- removed joint lbr_iiwa_joint_4
- removed joint lbr_iiwa_joint_5
- removed joint lbr_iiwa_joint_6
- removed joint lbr_iiwa_joint_7
