Commit message: URDF loading based on urdfdom for parsing and ASSIMP for collision objects meshes.

File: models/franka/dual_panda.urdf.xacro (robot description, xacro)
@@ -3,6 +3,6 @@
   <xacro:arg name="arm_id_1" default="panda_1" />
   <xacro:arg name="arm_id_2" default="panda_2" />
-  <xacro:include filename="$(find franka_description)/robots/panda_arm.xacro"/>
-  <xacro:include filename="$(find franka_description)/robots/hand.xacro"/>
+  <xacro:include filename="panda_arm.xacro"/>
+  <xacro:include filename="hand.xacro"/>
   <!-- box shaped table as base for the 2 Pandas -->
   <link name="base">

File: models/franka/panda.urdf.xacro (robot description, xacro)
@@ -10,9 +10,9 @@
   <xacro:arg name="hardware_interface" default="EffortJointInterface"/>
   <!-- Arm -->
-  <xacro:include filename="$(find franka_description)/robots/panda_arm.xacro"/>
+  <xacro:include filename="panda_arm.xacro"/>
   <xacro:panda_arm ns="$(arg robot_name)" connected_to="world" xyz="0 0 0" rpy="0 0 0" visual="true" collision="true" inertial="true" hardware_interface="EffortJointInterface" />
   <!-- Hand -->
   <xacro:if value="$(arg load_hand)">
-    <xacro:include filename="$(find franka_description)/robots/panda_hand.xacro"/>
+    <xacro:include filename="panda_hand.xacro"/>
     <xacro:panda_hand ns="$(arg robot_name)" connected_to="$(arg robot_name)_link8" xyz="0 0 0" rpy="0 0 ${-pi/4}" visual="true" collision="true" inertial="true" hardware_interface="EffortJointInterface"/>
   </xacro:if>

File: models/franka/panda_arm.xacro (robot description, xacro)
@@ -2,8 +2,8 @@
 <robot xmlns:xacro="http://www.ros.org/wiki/xacro" name="panda">
     <!-- Includes -->
-    <xacro:include filename="$(find franka_description)/robots/utils/panda_link.xacro" />
-    <xacro:include filename="$(find franka_description)/robots/utils/panda_joint.xacro" />
-    <xacro:include filename="$(find franka_description)/robots/utils/panda_transmission.xacro" />
-    <xacro:include filename="$(find franka_description)/robots/utils/panda_gazebo.xacro" />
+    <xacro:include filename="utils/panda_link.xacro" />
+    <xacro:include filename="utils/panda_joint.xacro" />
+    <xacro:include filename="utils/panda_transmission.xacro" />
+    <xacro:include filename="utils/panda_gazebo.xacro" />
     <!-- ns: Namespace of the panda. Serves to differentiate between arms in case of multiple instances. -->
     <xacro:macro name="panda_arm" params="ns:='panda' connected_to:='' xyz:='0 0 0' rpy:='0 0 0' visual:='true' collision:='true' inertial:='true' hardware_interface:=EffortJointInterface">

File: models/franka/panda_hand.xacro (robot description, xacro)
@@ -2,8 +2,8 @@
 <robot xmlns:xacro="http://www.ros.org/wiki/xacro" name="panda">
     <!-- Includes -->
-    <xacro:include filename="$(find franka_description)/robots/utils/panda_link.xacro" />
-    <xacro:include filename="$(find franka_description)/robots/utils/panda_joint.xacro" />
-    <xacro:include filename="$(find franka_description)/robots/utils/panda_transmission.xacro" />
-    <xacro:include filename="$(find franka_description)/robots/utils/panda_gazebo.xacro" />
+    <xacro:include filename="utils/panda_link.xacro" />
+    <xacro:include filename="utils/panda_joint.xacro" />
+    <xacro:include filename="utils/panda_transmission.xacro" />
+    <xacro:include filename="utils/panda_gazebo.xacro" />
     <!-- ns: Namespace of the panda. Serves to differentiate between arms in case of multiple instances. -->
     <xacro:macro name="panda_hand" params="ns:='panda' connected_to:='' xyz:='0 0 0' rpy:='0 0 0' visual:='true' collision:='true' inertial:='true' hardware_interface:=EffortJointInterface">

File: models/franka/utils/panda_link.xacro (robot description, xacro)
@@ -2,7 +2,7 @@
 <robot xmlns:xacro="http://www.ros.org/wiki/xacro" name="panda_link">
     <!-- Includes -->
-    <xacro:include filename="$(find franka_description)/robots/utils/panda_visual.xacro" />
-    <xacro:include filename="$(find franka_description)/robots/utils/panda_collision.xacro" />
-    <xacro:include filename="$(find franka_description)/robots/utils/panda_inertial.xacro" />
+    <xacro:include filename="panda_visual.xacro" />
+    <xacro:include filename="panda_collision.xacro" />
+    <xacro:include filename="panda_inertial.xacro" />
     <!-- Link -->
     <xacro:macro name="link" params="name visual:='' collision:='' inertial:='' *visual_block *collision_block *inertial_block">

File: models/iiwa/model.urdf (robot description, URDF)
Before this commit: robot lbr_iiwa, 3 links, 2 joints
Links:
- added link lbr_iiwa_link_3, mass 3; collision mesh filename=meshes/link_3.stl; visual mesh filename=meshes/link_3.obj
- added link lbr_iiwa_link_4, mass 2.7; collision mesh filename=meshes/link_4.stl; visual mesh filename=meshes/link_4.obj
- added link lbr_iiwa_link_5, mass 1.7; collision mesh filename=meshes/link_5.stl; visual mesh filename=meshes/link_5.obj
- added link lbr_iiwa_link_6, mass 1.8; collision mesh filename=meshes/link_6.stl; visual mesh filename=meshes/link_6.obj
- added link lbr_iiwa_link_7, mass 0.3; collision mesh filename=meshes/link_7.stl; visual mesh filename=meshes/link_7.obj
Joints:
- added joint lbr_iiwa_joint_3: type revolute, parent lbr_iiwa_link_2, child lbr_iiwa_link_3, origin xyz=0 0.2045 0 rpy=1.57079632679 0 3.14159265359, axis 0 0 1, limit lower=-2.96705972839 upper=2.96705972839 effort=300 velocity=10
- added joint lbr_iiwa_joint_4: type revolute, parent lbr_iiwa_link_3, child lbr_iiwa_link_4, origin xyz=0 0 0.2155 rpy=1.57079632679 0 0, axis 0 0 1, limit lower=-2.09439510239 upper=2.09439510239 effort=300 velocity=10
- added joint lbr_iiwa_joint_5: type revolute, parent lbr_iiwa_link_4, child lbr_iiwa_link_5, origin xyz=0 0.1845 0 rpy=-1.57079632679 3.14159265359 0, axis 0 0 1, limit lower=-2.96705972839 upper=2.96705972839 effort=300 velocity=10
- added joint lbr_iiwa_joint_6: type revolute, parent lbr_iiwa_link_5, child lbr_iiwa_link_6, origin xyz=0 0 0.2155 rpy=1.57079632679 0 0, axis 0 0 1, limit lower=-2.09439510239 upper=2.09439510239 effort=300 velocity=10
- added joint lbr_iiwa_joint_7: type revolute, parent lbr_iiwa_link_6, child lbr_iiwa_link_7, origin xyz=0 0.081 0 rpy=-1.57079632679 3.14159265359 0, axis 0 0 1, limit lower=-3.05432619099 upper=3.05432619099 effort=300 velocity=10
