Commit message: URDF loading and graphics fully working.

File: models/franka/panda_arm.xacro (robot description, xacro)
@@ -58,4 +58,5 @@
             <xacro:inertial mass="0.54" xyz="0.0109695 0.0107965 0.0650411" rpy="0 0 0" ixx="0.000888868887021" ixy="-0.00012239074652" ixz="3.98699829666e-05" iyy="0.000888001373233" iyz="-9.33825115206e-05" izz="0.0007176834609" />
         </xacro:link>
+        <!-- add default mass = 0, damping for prismatic joints and remove dummy link between arm and hand, visual rotation correction -->
         <link name="${ns}_link8"/>
         <!-- Joints -->

File: models/franka/urdf/panda.urdf (robot description, URDF)
Before this commit: robot panda, 13 links, 12 joints
Links:
- removed link panda_link8
- link panda_hand: geometry collision mesh filename=../meshes/collision/hand.stl; visual mesh filename=../meshes/visual/hand.dae
- link panda_leftfinger: geometry collision mesh filename=../meshes/collision/finger.stl; visual mesh filename=../meshes/visual/finger.dae
- link panda_link0: geometry collision mesh filename=../meshes/collision/link0.stl; visual mesh filename=../meshes/visual/link0.dae
- link panda_link1: geometry collision mesh filename=../meshes/collision/link1.stl; visual mesh filename=../meshes/visual/link1.dae
- link panda_link2: geometry collision mesh filename=../meshes/collision/link2.stl; visual mesh filename=../meshes/visual/link2.dae
- link panda_link3: geometry collision mesh filename=../meshes/collision/link3.stl; visual mesh filename=../meshes/visual/link3.dae
- link panda_link4: geometry collision mesh filename=../meshes/collision/link4.stl; visual mesh filename=../meshes/visual/link4.dae
- link panda_link5: geometry collision mesh filename=../meshes/collision/link5.stl; visual mesh filename=../meshes/visual/link5.dae
- link panda_link6: geometry collision mesh filename=../meshes/collision/link6.stl; visual mesh filename=../meshes/visual/link6.dae
- link panda_link7: geometry collision mesh filename=../meshes/collision/link7.stl; visual mesh filename=../meshes/visual/link7.dae
- link panda_rightfinger: geometry collision mesh filename=../meshes/collision/finger.stl; visual mesh filename=../meshes/visual/finger.dae
Joints:
- removed joint panda_joint8
- joint panda_hand_joint: origin xyz=0 0 0 rpy=0 0 -0.7853981633974483 -> xyz=0 0 0.107 rpy=0 0 -0.7853981633974483; parent panda_link8 -> panda_link7

File: models/iiwa/urdf/iiwa14.urdf (robot description, URDF)
Before this commit: robot iiwa14, 10 links, 9 joints
Links:
- link iiwa_link_0: geometry collision mesh filename=../meshes/iiwa14/collision/link_0.stl; visual mesh filename=../meshes/iiwa14/visual/link_0.stl
- link iiwa_link_1: geometry collision mesh filename=../meshes/iiwa14/collision/link_1.stl; visual mesh filename=../meshes/iiwa14/visual/link_1.stl
- link iiwa_link_2: geometry collision mesh filename=../meshes/iiwa14/collision/link_2.stl; visual mesh filename=../meshes/iiwa14/visual/link_2.stl
- link iiwa_link_3: geometry collision mesh filename=../meshes/iiwa14/collision/link_3.stl; visual mesh filename=../meshes/iiwa14/visual/link_3.stl
- link iiwa_link_4: geometry collision mesh filename=../meshes/iiwa14/collision/link_4.stl; visual mesh filename=../meshes/iiwa14/visual/link_4.stl
- link iiwa_link_5: geometry collision mesh filename=../meshes/iiwa14/collision/link_5.stl; visual mesh filename=../meshes/iiwa14/visual/link_5.stl
- link iiwa_link_6: geometry collision mesh filename=../meshes/iiwa14/collision/link_6.stl; visual mesh filename=../meshes/iiwa14/visual/link_6.stl
- link iiwa_link_7: geometry collision mesh filename=../meshes/iiwa14/collision/link_7.stl; visual mesh filename=../meshes/iiwa14/visual/link_7.stl
