Commit message: Started to adjust franka xacro.

File: models/franka/panda.urdf.xacro (robot description, xacro)
@@ -15,5 +15,5 @@
   <xacro:if value="$(arg load_hand)">
     <xacro:include filename="panda_hand.xacro"/>
-    <xacro:panda_hand ns="$(arg robot_name)" connected_to="$(arg robot_name)_link8" xyz="0 0 0" rpy="0 0 ${-pi/4}" visual="true" collision="true" inertial="true" hardware_interface="EffortJointInterface"/>
+    <xacro:panda_hand ns="$(arg robot_name)" connected_to="$(arg robot_name)_link7" xyz="0 0 0" rpy="0 0 ${-pi/4}" visual="true" collision="true" inertial="true" hardware_interface="EffortJointInterface"/>
   </xacro:if>
   <!-- Gazebo control plugin -->

File: models/franka/panda_arm.xacro (robot description, xacro)
@@ -17,5 +17,5 @@
             </joint>
         </xacro:unless>
-        <!-- Links  -->
+        <!-- Links -->
         <xacro:link name="link0" visual="${visual}" collision="${collision}" inertial="${inertial}">
             <xacro:visual xyz="${xyz}" rpy="${rpy}" mesh="link0" />
@@ -59,5 +59,5 @@
         </xacro:link>
         <!-- add default mass = 0, damping for prismatic joints and remove dummy link between arm and hand, visual rotation correction -->
-        <link name="${ns}_link8"/>
+        <!-- <link name="${ns}_link8"/> -->
         <!-- Joints -->
         <xacro:joint name="joint1" type="revolute" soft_lower_limit="-2.8973" soft_upper_limit="2.8973" rpy="0 0 0" xyz="0 0 0.333" parent="link0" child="link1" limit_effort="87" limit_lower="-2.8973" limit_upper="2.8973" limit_velocity="2.1750"/>
@@ -69,5 +69,5 @@
         <xacro:joint name="joint6" type="revolute" soft_lower_limit="-0.0175" soft_upper_limit="3.7525" rpy="${pi/2} 0 0" xyz="0 0 0" parent="link5" child="link6" limit_effort="12" limit_lower="-0.0175" limit_upper="3.7525" limit_velocity="2.6100"/>
         <xacro:joint name="joint7" type="revolute" soft_lower_limit="-2.8973" soft_upper_limit="2.8973" rpy="${pi/2} 0 0" xyz="0.088 0 0" parent="link6" child="link7" limit_effort="12" limit_lower="-2.8973" limit_upper="2.8973" limit_velocity="2.6100"/>
-        <xacro:joint name="joint8" type="fixed" parent="link7" child="link8" rpy="0 0 0" xyz="0 0 0.107"/>
+        <!-- <xacro:joint name="joint8" type="fixed" parent="link7" child="link8" rpy="0 0 0" xyz="0 0 0.107"/> -->
         <!-- Transmissions -->
         <xacro:transmission name="tran1" joint="joint1" motor="motor1" hardware_interface="${hardware_interface}" />

File: models/franka/panda_hand.xacro (robot description, xacro)
@@ -13,5 +13,5 @@
                 <parent link="${connected_to}"/>
                 <child link="${ns}_hand"/>
-                <origin xyz="${xyz}" rpy="${rpy}"/>
+                <origin xyz="${xyz}" rpy="${rpy}"/> <!--0.107-->
             </joint>
         </xacro:unless>
@@ -39,4 +39,5 @@
             <axis xyz="0 1 0"/>
             <limit effort="20" lower="-0.001" upper="0.04" velocity="0.3"/>
+            <dynamics damping="0.5"/>
         </joint>
         <joint name="${ns}_finger_joint2" type="prismatic">
@@ -46,4 +47,5 @@
             <axis xyz="0 -1 0"/>
             <limit effort="20" lower="-0.001" upper="0.04" velocity="0.3"/>
+            <dynamics damping="0.5"/>
         </joint>
         <!-- Transmissions -->

File: models/franka/utils/panda_visual.xacro (robot description, xacro)
@@ -1,5 +1,5 @@
 <?xml version='1.0' encoding='utf-8'?>
 <robot xmlns:xacro="http://www.ros.org/wiki/xacro" name="panda_visual">
-    <xacro:macro name="visual" params="xyz:='0 0 0' rpy:='0 0 0' mesh:=''">
+    <xacro:macro name="visual" params="xyz:='1.57079632679 0 0' rpy:='0 0 0' mesh:=''">
         <visual>
             <origin xyz="${xyz}" rpy="${rpy}"/>
