Commit message: Added some model and compiled the urdf from xacro.

File: models/franka/utils/panda_collision.xacro (robot description, xacro)
@@ -5,5 +5,5 @@
             <origin xyz="${xyz}" rpy="${rpy}"/>
             <geometry>
-                <mesh filename="package://franka_description/robots/meshes/collision/${mesh}.stl"/>
+                <mesh filename="meshes/collision/${mesh}.stl"/>
             </geometry>
         </collision>

File: models/franka/utils/panda_visual.xacro (robot description, xacro)
@@ -5,5 +5,5 @@
             <origin xyz="${xyz}" rpy="${rpy}"/>
             <geometry>
-                <mesh filename="package://franka_description/robots/meshes/visual/${mesh}.dae"/>
+                <mesh filename="meshes/visual/${mesh}.dae"/>
             </geometry>
         </visual>
